File: Hardware/DualTrackingSupply.sch (KiCad schematic (older format))
At the start: 0 parts

Commit message: Basic regulator topology
Parts:
- added B?: GBU806, symbol RECT-BRIDGE
- added C? (x4): CP, ~, symbol CP
- added C? (x4): 0.1uF, ~, symbol C
- added C? (x2): 10uF, ~, symbol CP
- added D? (x4): 1N4004, ~, symbol DIODE
- added J?: IN, ~, symbol CONN-3
- added J?: OUT, ~, symbol CONN-3
- added R? (x2): 100, ~, symbol R
- added R? (x2): 5k, ~, symbol R
- added RV?: 5k, ~, symbol POT
- added U?: LM317, symbol LDO-3
- added U?: LM337, symbol LDO-NEG-3
Connections:
- new net: C?.1, D?.1, R?.1, R?.2, RV?.3, U?.1 (Adj)
- new net: C?.1, C?.1, D?.1, D?.2, J?.1, R?.2, U?.2 (Out)
- new net: B?.1 (+), C?.1, C?.1, D?.2, U?.3 (In)
- new net: C?.2, D?.2, R?.1, R?.2, RV?.1, RV?.2, U?.1 (Adj)
- new net: B?.4 (-), C?.2, C?.2, D?.1, U?.2 (In)
- new net: C?.2, C?.2, D?.1, D?.2, J?.3, R?.1, U?.3 (Out)
- new net: B?.2, J?.1
- new net: B?.3, J?.3
- new net GND: C?.1, C?.1, C?.1, C?.1, C?.1, C?.2, C?.2, C?.2, C?.2, C?.2, J?.2, J?.2, R?.1, R?.2
Other:
- note added: "Hammond\n166M25\nTransformer"
